Commit message: succeed in visualization

File: urdf/gem/urdf/gem.urdf (robot description, URDF)
Before this commit: robot gem, 40 links, 39 joints
Links:
- link base_link: geometry collision mesh filename=../meshes/base_link.STL; visual mesh filename=../meshes/base_link.STL
- link chair_link: geometry collision mesh filename=../meshes/chair_link.STL; visual mesh filename=../meshes/chair_link.STL
- link door_link: geometry collision mesh filename=../meshes/door_link.STL; visual mesh filename=../meshes/door_link.STL
- link front_camera_link: geometry collision mesh filename=../meshes/front_camera_link.STL; visual mesh filename=../meshes/front_camera_link.STL
- link front_left_emergency_button_link: geometry collision mesh filename=../meshes/front_left_emergency_button_link.STL; visual mesh filename=../meshes/front_left_emergency_button_link.STL
- link front_left_head_light_link: geometry collision mesh filename=../meshes/front_left_head_light_link.STL; visual mesh filename=../meshes/front_left_head_light_link.STL
- link front_left_turn_light_link: geometry collision mesh filename=../meshes/front_left_turn_light_link.STL; visual mesh filename=../meshes/front_left_turn_light_link.STL
- link front_left_wheel_link: geometry collision sphere radius=0.295; visual mesh filename=../meshes/front_left_wheel_link.STL
- link front_rack_link: geometry collision mesh filename=../meshes/front_rack_link.STL; visual mesh filename=../meshes/front_rack_link.STL
- link front_right_emergency_button_link: geometry collision mesh filename=../meshes/front_right_emergency_button_link.STL; visual mesh filename=../meshes/front_right_emergency_button_link.STL
- link front_right_head_light_link: geometry collision mesh filename=../meshes/front_right_head_light_link.STL; visual mesh filename=../meshes/front_right_head_light_link.STL
- link front_right_turn_light_link: geometry collision mesh filename=../meshes/front_right_turn_light_link.STL; visual mesh filename=../meshes/front_right_turn_light_link.STL
- link front_right_wheel_link: geometry collision sphere radius=0.295; visual mesh filename=../meshes/front_right_wheel_link.STL
- link left_I_link: geometry collision mesh filename=../meshes/left_I_link.STL; visual mesh filename=../meshes/left_I_link.STL
- link left_antenna_link: geometry collision mesh filename=../meshes/left_antenna_link.STL; visual mesh filename=../meshes/left_antenna_link.STL
- link left_blue_outer_link: geometry collision mesh filename=../meshes/left_blue_outer_link.STL; visual mesh filename=../meshes/left_blue_outer_link.STL
- link rear_left_emergency_button_link: geometry collision mesh filename=../meshes/rear_left_emergency_button_link.STL; visual mesh filename=../meshes/rear_left_emergency_button_link.STL
- link rear_left_light_link: geometry collision mesh filename=../meshes/rear_left_light_link.STL; visual mesh filename=../meshes/rear_left_light_link.STL
- link rear_left_stop_light_link: geometry collision mesh filename=../meshes/rear_left_stop_light_link.STL; visual mesh filename=../meshes/rear_left_stop_light_link.STL
- link rear_left_wheel_link: geometry collision sphere radius=0.295; visual mesh filename=../meshes/rear_left_wheel_link.STL
- link rear_light_bar_link: geometry collision mesh filename=../meshes/rear_light_bar_link.STL; visual mesh filename=../meshes/rear_light_bar_link.STL
- link rear_rack_link: geometry collision mesh filename=../meshes/rear_rack_link.STL; visual mesh filename=../meshes/rear_rack_link.STL
- link rear_right_emergency_button_link: geometry collision mesh filename=../meshes/rear_right_emergency_button_link.STL; visual mesh filename=../meshes/rear_right_emergency_button_link.STL
- link rear_right_light_link: geometry collision mesh filename=../meshes/rear_right_light_link.STL; visual mesh filename=../meshes/rear_right_light_link.STL
- link rear_right_stop_light_link: geometry collision mesh filename=../meshes/rear_right_stop_light_link.STL; visual mesh filename=../meshes/rear_right_stop_light_link.STL
- link rear_right_wheel_link: geometry collision sphere radius=0.295; visual mesh filename=../meshes/rear_right_wheel_link.STL
- link right_I_link: geometry collision mesh filename=../meshes/right_I_link.STL; visual mesh filename=../meshes/right_I_link.STL
- link right_antenna_link: geometry collision mesh filename=../meshes/right_antenna_link.STL; visual mesh filename=../meshes/right_antenna_link.STL
- link right_blue_outer_link: geometry collision mesh filename=../meshes/right_blue_outer_link.STL; visual mesh filename=../meshes/right_blue_outer_link.STL
- link top_rack_link: geometry collision mesh filename=../meshes/top_rack_link.STL; visual mesh filename=../meshes/top_rack_link.STL
- link velodyne: geometry visual mesh filename=../meshes/VLP16_scan.stl
- link velodyne_base_link: geometry collision cylinder length=0.0717 radius=0.0516; visual mesh filename=../meshes/VLP16_base_1.stl
